Commit message: Thrusters are now a macro

File: urdf/spaceship.urdf.xacro (robot description, xacro)
@@ -1,8 +1,6 @@
 <robot xmlns:xacro="http://www.ros.org/wiki/xacro" name="tie_fighter">
+ <xacro:include filename="$(find gazebo_spaceship)/urdf/thruster.urdf.xacro"/>
     <material name="white">
       <color rgba="1 1 1 1"/>
-    </material>
-    <material name="black">
-      <color rgba="0 0 0 1"/>
     </material>
     <link name="base_link">
@@ -40,31 +38,21 @@
       </inertia>
     </link>-->
-    <link name="top_thruster_link">
-      <visual>
-        <geometry>
-          <box size="0.1 0.1 0.3"/>
-        </geometry>
-        <origin xyz="0 0 1.3"/>
-        <material name="black"/>
-      </visual>
-    </link>
+    <link name="top_thruster_link"/>
     <joint name="top_thruster_joint" type="fixed" >
       <parent link="base_link" />
       <child link="top_thruster_link" />
-      <origin xyz="0 0 0" rpy="0 0 0"/>
+      <origin xyz="0 0 -1.3" rpy="0 0 0"/>
     </joint>
-    <link name="bottom_thruster_link">
-      <visual>
-        <geometry>
-          <box size="1 1 0.3"/>
-        </geometry>
-        <origin xyz="0 0 -1.3"/>
-        <material name="black"/>
-      </visual>
-    </link>
+    <xacro:thruster name="top_thruster" parent="top_thruster_link">
+      <origin xyz="0 0 0" rpy="0 0 0" />
+    </xacro:thruster>
+    <link name="bottom_thruster_link"/>
     <joint name="bottom_thruster_joint" type="fixed" >
       <parent link="base_link" />
       <child link="bottom_thruster_link" />
-      <origin xyz="0 0 0" rpy="0 0 0"/>
+      <origin xyz="0 0 -1.3" rpy="0 0 0"/>
     </joint>
+    <xacro:thruster name="bottom_thruster" parent="bottom_thruster_link">
+      <origin xyz="0 0 0" rpy="0 0 0" />
+    </xacro:thruster>
 </robot>

Commit message: Visible in gazebo too, added some thrusters but I think I need some more for pitching

File: urdf/spaceship.urdf.xacro (robot description, xacro)
@@ -1,2 +1,3 @@
+<?xml version="1.0"?>
 <robot xmlns:xacro="http://www.ros.org/wiki/xacro" name="tie_fighter">
  <xacro:include filename="$(find gazebo_spaceship)/urdf/thruster.urdf.xacro"/>
@@ -16,31 +17,22 @@
         </geometry>
       </collision>
-      <inertia>
-         <mass value="10.0"/>
-         <inertia ixx="0.000002" ixy="0.0" ixz="0.0" iyy="0.000001" iyz="0.0" izz="0.000002"/>
-      </inertia>
+      <!-- <collision>
+        <geometry>
+          <box size="8 6 10"/>
+        </geometry>
+      </collision> -->
+      <inertial>
+         <mass value="1.0"/>
+         <inertia
+        ixx="1.0" ixy="0.0" ixz="0.0"
+        iyy="1.0" iyz="0.0"
+        izz="1.0"/>
+      </inertial>
     </link>
-    <!-- <link name="base_link">
-      <visual>
-        <geometry>
-          <box size="2 2 2" />
-        </geometry>
-        <material name="white"/>
-      </visual>
-      <collision>
-        <geometry>
-          <box size="2 2 2" />
-        </geometry>
-      </collision>
-      <inertia>
-         <mass value="10.0"/>
-         <inertia ixx="0.000002" ixy="0.0" ixz="0.0" iyy="0.000001" iyz="0.0" izz="0.000002"/>
-      </inertia>
-    </link>-->
     <link name="top_thruster_link"/>
     <joint name="top_thruster_joint" type="fixed" >
       <parent link="base_link" />
       <child link="top_thruster_link" />
-      <origin xyz="0 0 -1.3" rpy="0 0 0"/>
+      <origin xyz="0 0 1.4" rpy="0 0 0"/>
     </joint>
     <xacro:thruster name="top_thruster" parent="top_thruster_link">
@@ -51,8 +43,101 @@
       <parent link="base_link" />
       <child link="bottom_thruster_link" />
-      <origin xyz="0 0 -1.3" rpy="0 0 0"/>
+      <origin xyz="0 0 -1.4" rpy="${pi} 0 0"/>
     </joint>
     <xacro:thruster name="bottom_thruster" parent="bottom_thruster_link">
       <origin xyz="0 0 0" rpy="0 0 0" />
     </xacro:thruster>
+    <link name="front_thruster_link"/>
+    <joint name="front_thruster_joint" type="fixed" >
+      <parent link="base_link" />
+      <child link="front_thruster_link" />
+      <origin xyz="0 1.4 0" rpy="${-pi/2} 0 0"/>
+    </joint>
+    <xacro:thruster name="front_thruster" parent="front_thruster_link">
+      <origin xyz="0 0 0" rpy="0 0 0" />
+    </xacro:thruster>
+    <link name="back_thruster_link"/>
+    <joint name="back_thruster_joint" type="fixed" >
+      <parent link="base_link" />
+      <child link="back_thruster_link" />
+      <origin xyz="0 -1.4 0" rpy="${pi/2} 0 0"/>
+    </joint>
+    <xacro:thruster name="back_thruster" parent="back_thruster_link">
+      <origin xyz="0 0 0" rpy="0 0 0" />
+    </xacro:thruster>
+    <link name="top_left_front_thruster_link"/>
+    <joint name="top_left_front_thruster_joint" type="fixed" >
+      <parent link="base_link" />
+      <child link="top_left_front_thruster_link" />
+      <origin xyz="3.85 3 4.5" rpy="0 ${pi/2} 0"/>
+    </joint>
+    <xacro:thruster name="top_left_front_thruster" parent="top_left_front_thruster_link">
+      <origin xyz="0 0 0" rpy="0 0 0" />
+    </xacro:thruster>
+    <link name="top_left_back_thruster_link"/>
+    <joint name="top_left_back_thruster_joint" type="fixed" >
+      <parent link="base_link" />
+      <child link="top_left_back_thruster_link" />
+      <origin xyz="3.85 -3 4.5" rpy="0 ${pi/2} 0"/>
+    </joint>
+    <xacro:thruster name="top_left_back_thruster" parent="top_left_back_thruster_link">
+      <origin xyz="0 0 0" rpy="0 0 0" />
+    </xacro:thruster>
+    <link name="bottom_left_front_thruster_link"/>
+    <joint name="bottom_left_front_thruster_joint" type="fixed" >
+      <parent link="base_link" />
+      <child link="bottom_left_front_thruster_link" />
+      <origin xyz="3.85 3 -4.5" rpy="0 ${pi/2} 0"/>
+    </joint>
+    <xacro:thruster name="bottom_left_front_thruster" parent="bottom_left_front_thruster_link">
+      <origin xyz="0 0 0" rpy="0 0 0" />
+    </xacro:thruster>
+    <link name="bottom_left_back_thruster_link"/>
+    <joint name="bottom_left_back_thruster_joint" type="fixed" >
+      <parent link="base_link" />
+      <child link="bottom_left_back_thruster_link" />
+      <origin xyz="3.85 -3 -4.5" rpy="0 ${pi/2} 0"/>
+    </joint>
+    <xacro:thruster name="bottom_left_back_thruster" parent="bottom_left_back_thruster_link">
+      <origin xyz="0 0 0" rpy="0 0 0" />
+    </xacro:thruster>
+    <link name="top_right_front_thruster_link"/>
+    <joint name="top_right_front_thruster_joint" type="fixed" >
+      <parent link="base_link" />
+      <child link="top_right_front_thruster_link" />
+      <origin xyz="-3.85 3 4.5" rpy="0 ${-pi/2} 0"/>
+    </joint>
+    <xacro:thruster name="top_right_front_thruster" parent="top_right_front_thruster_link">
+      <origin xyz="0 0 0" rpy="0 0 0" />
+    </xacro:thruster>
+    <link name="top_right_back_thruster_link"/>
+    <joint name="top_right_back_thruster_joint" type="fixed" >
+      <parent link="base_link" />
+      <child link="top_right_back_thruster_link" />
+      <origin xyz="-3.85 -3 4.5" rpy="0 ${-pi/2} 0"/>
+    </joint>
+    <xacro:thruster name="top_right_back_thruster" parent="top_right_back_thruster_link">
+      <origin xyz="0 0 0" rpy="0 0 0" />
+    </xacro:thruster>
+    <link name="bottom_right_front_thruster_link"/>
+    <joint name="bottom_right_front_thruster_joint" type="fixed" >
+      <parent link="base_link" />
+      <child link="bottom_right_front_thruster_link" />
+      <origin xyz="-3.85 3 -4.5" rpy="0 ${-pi/2} 0"/>
+    </joint>
+    <xacro:thruster name="bottom_right_front_thruster" parent="bottom_right_front_thruster_link">
+      <origin xyz="0 0 0" rpy="0 0 0" />
+    </xacro:thruster>
+    <link name="bottom_right_back_thruster_link"/>
+    <joint name="bottom_right_back_thruster_joint" type="fixed" >
+      <parent link="base_link" />
+      <child link="bottom_right_back_thruster_link" />
+      <origin xyz="-3.85 -3 -4.5" rpy="0 ${-pi/2} 0"/>
+    </joint>
+    <xacro:thruster name="bottom_right_back_thruster" parent="bottom_right_back_thruster_link">
+      <origin xyz="0 0 0" rpy="0 0 0" />
+    </xacro:thruster>
+    <gazebo reference="base_link">
+      <material>Gazebo/White</material>
+    </gazebo>
 </robot>

File: urdf/thruster.urdf.xacro (robot description, xacro)
@@ -15,4 +15,13 @@
       </visual>
     </link>
+   <!--  <gazebo>
+      <plugin name="${name}_propulsion" filename="libthruster_ros_plugin.so">
+       <linkName>${namespace}/thruster_${thruster_id}</linkName>
+        <jointName>${namespace}/thruster_${thruster_id}_joint</jointName>
+        <thrusterID>${thruster_id}</thrusterID>
+        <xacro:insert_block name="dynamics"/>
+        <xacro:insert_block name="conversion"/>
+      </plugin>
+    </gazebo> -->
   </xacro:macro>
 </robot>

Commit message: Added uuv thrusters. Not working yet, but the topics are available

File: urdf/spaceship.urdf.xacro (robot description, xacro)
@@ -17,9 +17,4 @@
         </geometry>
       </collision>
-      <!-- <collision>
-        <geometry>
-          <box size="8 6 10"/>
-        </geometry>
-      </collision> -->
       <inertial>
          <mass value="1.0"/>
@@ -30,114 +25,48 @@
       </inertial>
     </link>
-    <link name="top_thruster_link"/>
-    <joint name="top_thruster_joint" type="fixed" >
-      <parent link="base_link" />
-      <child link="top_thruster_link" />
+    <xacro:thruster name="top_thruster" thruster_id="0">
       <origin xyz="0 0 1.4" rpy="0 0 0"/>
-    </joint>
-    <xacro:thruster name="top_thruster" parent="top_thruster_link">
-      <origin xyz="0 0 0" rpy="0 0 0" />
     </xacro:thruster>
-    <link name="bottom_thruster_link"/>
-    <joint name="bottom_thruster_joint" type="fixed" >
-      <parent link="base_link" />
-      <child link="bottom_thruster_link" />
+    <xacro:thruster name="bottom_thruster" thruster_id="1">
       <origin xyz="0 0 -1.4" rpy="${pi} 0 0"/>
-    </joint>
-    <xacro:thruster name="bottom_thruster" parent="bottom_thruster_link">
-      <origin xyz="0 0 0" rpy="0 0 0" />
     </xacro:thruster>
-    <link name="front_thruster_link"/>
-    <joint name="front_thruster_joint" type="fixed" >
-      <parent link="base_link" />
-      <child link="front_thruster_link" />
+    <xacro:thruster name="front_thruster" thruster_id="2">
       <origin xyz="0 1.4 0" rpy="${-pi/2} 0 0"/>
-    </joint>
-    <xacro:thruster name="front_thruster" parent="front_thruster_link">
-      <origin xyz="0 0 0" rpy="0 0 0" />
     </xacro:thruster>
-    <link name="back_thruster_link"/>
-    <joint name="back_thruster_joint" type="fixed" >
-      <parent link="base_link" />
-      <child link="back_thruster_link" />
+    <xacro:thruster name="back_thruster" thruster_id="3">
       <origin xyz="0 -1.4 0" rpy="${pi/2} 0 0"/>
-    </joint>
-    <xacro:thruster name="back_thruster" parent="back_thruster_link">
-      <origin xyz="0 0 0" rpy="0 0 0" />
     </xacro:thruster>
-    <link name="top_left_front_thruster_link"/>
-    <joint name="top_left_front_thruster_joint" type="fixed" >
-      <parent link="base_link" />
-      <child link="top_left_front_thruster_link" />
+    <xacro:thruster name="top_left_front_thruster" thruster_id="4">
       <origin xyz="3.85 3 4.5" rpy="0 ${pi/2} 0"/>
-    </joint>
-    <xacro:thruster name="top_left_front_thruster" parent="top_left_front_thruster_link">
-      <origin xyz="0 0 0" rpy="0 0 0" />
     </xacro:thruster>
-    <link name="top_left_back_thruster_link"/>
-    <joint name="top_left_back_thruster_joint" type="fixed" >
-      <parent link="base_link" />
-      <child link="top_left_back_thruster_link" />
+    <xacro:thruster name="top_left_back_thruster" thruster_id="5">
       <origin xyz="3.85 -3 4.5" rpy="0 ${pi/2} 0"/>
-    </joint>
-    <xacro:thruster name="top_left_back_thruster" parent="top_left_back_thruster_link">
-      <origin xyz="0 0 0" rpy="0 0 0" />
     </xacro:thruster>
-    <link name="bottom_left_front_thruster_link"/>
-    <joint name="bottom_left_front_thruster_joint" type="fixed" >
-      <parent link="base_link" />
-      <child link="bottom_left_front_thruster_link" />
+    <xacro:thruster name="bottom_left_front_thruster" thruster_id="6">
       <origin xyz="3.85 3 -4.5" rpy="0 ${pi/2} 0"/>
-    </joint>
-    <xacro:thruster name="bottom_left_front_thruster" parent="bottom_left_front_thruster_link">
-      <origin xyz="0 0 0" rpy="0 0 0" />
     </xacro:thruster>
-    <link name="bottom_left_back_thruster_link"/>
-    <joint name="bottom_left_back_thruster_joint" type="fixed" >
-      <parent link="base_link" />
-      <child link="bottom_left_back_thruster_link" />
+    <xacro:thruster name="bottom_left_back_thruster" thruster_id="7">
       <origin xyz="3.85 -3 -4.5" rpy="0 ${pi/2} 0"/>
-    </joint>
-    <xacro:thruster name="bottom_left_back_thruster" parent="bottom_left_back_thruster_link">
-      <origin xyz="0 0 0" rpy="0 0 0" />
     </xacro:thruster>
-    <link name="top_right_front_thruster_link"/>
-    <joint name="top_right_front_thruster_joint" type="fixed" >
-      <parent link="base_link" />
-      <child link="top_right_front_thruster_link" />
+    <xacro:thruster name="top_right_front_thruster" thruster_id="8">
       <origin xyz="-3.85 3 4.5" rpy="0 ${-pi/2} 0"/>
-    </joint>
-    <xacro:thruster name="top_right_front_thruster" parent="top_right_front_thruster_link">
-      <origin xyz="0 0 0" rpy="0 0 0" />
     </xacro:thruster>
-    <link name="top_right_back_thruster_link"/>
-    <joint name="top_right_back_thruster_joint" type="fixed" >
-      <parent link="base_link" />
-      <child link="top_right_back_thruster_link" />
+    <xacro:thruster name="top_right_back_thruster" thruster_id="9">
       <origin xyz="-3.85 -3 4.5" rpy="0 ${-pi/2} 0"/>
-    </joint>
-    <xacro:thruster name="top_right_back_thruster" parent="top_right_back_thruster_link">
-      <origin xyz="0 0 0" rpy="0 0 0" />
     </xacro:thruster>
-    <link name="bottom_right_front_thruster_link"/>
-    <joint name="bottom_right_front_thruster_joint" type="fixed" >
-      <parent link="base_link" />
-      <child link="bottom_right_front_thruster_link" />
+    <xacro:thruster name="bottom_right_front_thruster" thruster_id="10">
       <origin xyz="-3.85 3 -4.5" rpy="0 ${-pi/2} 0"/>
-    </joint>
-    <xacro:thruster name="bottom_right_front_thruster" parent="bottom_right_front_thruster_link">
-      <origin xyz="0 0 0" rpy="0 0 0" />
     </xacro:thruster>
-    <link name="bottom_right_back_thruster_link"/>
-    <joint name="bottom_right_back_thruster_joint" type="fixed" >
-      <parent link="base_link" />
-      <child link="bottom_right_back_thruster_link" />
+    <xacro:thruster name="bottom_right_back_thruster" thruster_id="11">
       <origin xyz="-3.85 -3 -4.5" rpy="0 ${-pi/2} 0"/>
-    </joint>
-    <xacro:thruster name="bottom_right_back_thruster" parent="bottom_right_back_thruster_link">
-      <origin xyz="0 0 0" rpy="0 0 0" />
     </xacro:thruster>
     <gazebo reference="base_link">
       <material>Gazebo/White</material>
     </gazebo>
+    <gazebo>
+    <plugin name="joint_state_publisher" filename="libjoint_state_publisher.so">
+      <robotNamespace></robotNamespace>
+      <updateRate>50</updateRate>
+    </plugin>
+  </gazebo>
 </robot>

File: urdf/thruster.urdf.xacro (robot description, xacro)
@@ -1,10 +1,5 @@
 <?xml version="1.0"?>
 <robot xmlns:xacro="http://www.ros.org/wiki/xacro">
-  <xacro:macro name="thruster" params="parent name *origin ">
-    <joint name="${name}_base_joint" type="fixed" >
-      <parent link="${parent}" />
-      <child link="${name}_base_link" />
-      <xacro:insert_block name="origin" />
-    </joint>
+  <xacro:macro name="thruster" params="name thruster_id *origin ">
     <link name="${name}_base_link">
       <visual>
@@ -14,14 +9,89 @@
         <material name="black"/>
       </visual>
+      <inertial>
+        <mass value="0.001" />
+        <origin xyz="0 0 0" rpy="0 0 0"/>
+        <inertia ixx="0.000000017" ixy="0.0" ixz="0.0"
+               iyy="0.000000017" iyz="0.0"
+               izz="0.000000017" />
+      </inertial>
     </link>
-   <!--  <gazebo>
-      <plugin name="${name}_propulsion" filename="libthruster_ros_plugin.so">
-       <linkName>${namespace}/thruster_${thruster_id}</linkName>
-        <jointName>${namespace}/thruster_${thruster_id}_joint</jointName>
-        <thrusterID>${thruster_id}</thrusterID>
-        <xacro:insert_block name="dynamics"/>
-        <xacro:insert_block name="conversion"/>
+    <joint name="${name}_joint" type="continuous" >
+      <parent link="base_link" />
+      <child link="${name}_base_link" />
+      <xacro:insert_block name="origin" />
+    </joint>
+    <gazebo>
+      <!-- Thruster ROS plugin -->
+      <plugin name="${name}_thruster_model" filename="libthruster_ros_plugin.so">
+        <!-- Name of the thruster link -->
+        <linkName>${name}_base_link</linkName>
+        <!-- Name of the joint between thruster and vehicle base link -->
+        <jointName>${name}_joint</jointName>
+         <thrusterID>${thruster_id}</thrusterID>
+        <!-- Thruster force output topic name -->
+        <thrustTopic>/thrusters/${name}/thrust</thrustTopic>
+        <!-- Thruster commmand input topic name -->
+        <inputTopic>/thrusters/${name}/input</inputTopic>
+        <!-- Gain of the input command signal -->
+        <gain>1</gain>
+        <!-- Maximum allowed input value for the input signal for thruster unit -->
+        <clampMax>0</clampMax>
+        <!-- Minimum allowed value for the input signal for thruster unit -->
+        <clampMin>0</clampMin>
+        <!--
+        Value from 0 to 1 to set the efficiency of the output thrust force
+        Default value is 1.0
+        -->
+        <thrust_efficiency>1</thrust_efficiency>
+        <!--
+        Value from 0 to 1 to set the efficiency of the propeller as a factor
+        to be multiplied to the current value of the state variable at each
+        iteration.
+        Default value is 1.0
+        -->
+        <propeller_efficiency>1</propeller_efficiency>
+        <!-- Simple zero-order model -->
+        <dynamics>
+          <type>ZeroOrder</type>
+        </dynamics>
+        <!-- <dynamics>
+          <type>FirstOrder</type>
+          <timeConstant>0.0</timeConstant>
+        </dynamics>
+        <dynamics>
+          <type>Yoerger</type>
+          <alpha>0.0</alpha>
+          <beta>0.0</beta>
+        </dynamics>
+        <dynamics>
+          <type>Bessa</type>
+          <Jmsp>0.0</Jmsp>
+          <Kv1>0.0</Kv1>
+          <Kv2>0.0</Kv2>
+          <Kt>0.0</Kt>
+          <Rm>0.0</Rm>
+        </dynamics> -->
+        <conversion>
+          <type>Basic</type>
+          <rotorConstant>0.0</rotorConstant>
+        </conversion>
+        <!-- <conversion>
+          <type>Bessa</type>
+          <rotorConstantL>0.0</rotorConstantL>
+          <rotorConstantR>0.0</rotorConstantR>
+          <deltaL>0.0</deltaL>
+          <deltaR>0.0</deltaR>
+        </conversion>
+        <conversion>
+          <type>LinearInterp</type>
+          <inputValues>0 1 2 3</inputValues>
+          <outputValues>0 1 2 3</outputValues>
+        </conversion> -->
       </plugin>
-    </gazebo> -->
+    </gazebo>
+    <gazebo reference="thruster_${name}">
+      <selfCollide>false</selfCollide>
+    </gazebo>
   </xacro:macro>
 </robot>
