Commit message: Using my custom air thruster plugin, and it seems to be working!

File: urdf/spaceship.urdf.xacro (robot description, xacro)
@@ -25,38 +25,38 @@
       </inertial>
     </link>
-    <xacro:thruster name="top_thruster" thruster_id="0">
+    <xacro:thruster name="top_thruster" thruster_name="0">
       <origin xyz="0 0 1.4" rpy="0 0 0"/>
     </xacro:thruster>
-    <xacro:thruster name="bottom_thruster" thruster_id="1">
+    <xacro:thruster name="bottom_thruster" thruster_name="1">
       <origin xyz="0 0 -1.4" rpy="${pi} 0 0"/>
     </xacro:thruster>
-    <xacro:thruster name="front_thruster" thruster_id="2">
+    <xacro:thruster name="front_thruster" thruster_name="2">
       <origin xyz="0 1.4 0" rpy="${-pi/2} 0 0"/>
     </xacro:thruster>
-    <xacro:thruster name="back_thruster" thruster_id="3">
+    <xacro:thruster name="back_thruster" thruster_name="3">
       <origin xyz="0 -1.4 0" rpy="${pi/2} 0 0"/>
     </xacro:thruster>
-    <xacro:thruster name="top_left_front_thruster" thruster_id="4">
+    <xacro:thruster name="top_left_front_thruster" thruster_name="4">
       <origin xyz="3.85 3 4.5" rpy="0 ${pi/2} 0"/>
     </xacro:thruster>
-    <xacro:thruster name="top_left_back_thruster" thruster_id="5">
+    <xacro:thruster name="top_left_back_thruster" thruster_name="5">
       <origin xyz="3.85 -3 4.5" rpy="0 ${pi/2} 0"/>
     </xacro:thruster>
-    <xacro:thruster name="bottom_left_front_thruster" thruster_id="6">
+    <xacro:thruster name="bottom_left_front_thruster" thruster_name="6">
       <origin xyz="3.85 3 -4.5" rpy="0 ${pi/2} 0"/>
     </xacro:thruster>
-    <xacro:thruster name="bottom_left_back_thruster" thruster_id="7">
+    <xacro:thruster name="bottom_left_back_thruster" thruster_name="7">
       <origin xyz="3.85 -3 -4.5" rpy="0 ${pi/2} 0"/>
     </xacro:thruster>
-    <xacro:thruster name="top_right_front_thruster" thruster_id="8">
+    <xacro:thruster name="top_right_front_thruster" thruster_name="8">
       <origin xyz="-3.85 3 4.5" rpy="0 ${-pi/2} 0"/>
     </xacro:thruster>
-    <xacro:thruster name="top_right_back_thruster" thruster_id="9">
+    <xacro:thruster name="top_right_back_thruster" thruster_name="9">
       <origin xyz="-3.85 -3 4.5" rpy="0 ${-pi/2} 0"/>
     </xacro:thruster>
-    <xacro:thruster name="bottom_right_front_thruster" thruster_id="10">
+    <xacro:thruster name="bottom_right_front_thruster" thruster_name="10">
       <origin xyz="-3.85 3 -4.5" rpy="0 ${-pi/2} 0"/>
     </xacro:thruster>
-    <xacro:thruster name="bottom_right_back_thruster" thruster_id="11">
+    <xacro:thruster name="bottom_right_back_thruster" thruster_name="11">
       <origin xyz="-3.85 -3 -4.5" rpy="0 ${-pi/2} 0"/>
     </xacro:thruster>

File: urdf/thruster.urdf.xacro (robot description, xacro)
@@ -1,5 +1,5 @@
 <?xml version="1.0"?>
 <robot xmlns:xacro="http://www.ros.org/wiki/xacro">
-  <xacro:macro name="thruster" params="name thruster_id *origin ">
+  <xacro:macro name="thruster" params="name thruster_name *origin ">
     <link name="${name}_base_link">
       <visual>
@@ -23,70 +23,8 @@
     </joint>
     <gazebo>
-      <!-- Thruster ROS plugin -->
-      <plugin name="${name}_thruster_model" filename="libthruster_ros_plugin.so">
-        <!-- Name of the thruster link -->
+      <plugin name="${name}_thruster_model" filename="libair_thruster_ros_plugin.so">
         <linkName>${name}_base_link</linkName>
-        <!-- Name of the joint between thruster and vehicle base link -->
-        <jointName>${name}_joint</jointName>
-         <thrusterID>${thruster_id}</thrusterID>
-        <!-- Thruster force output topic name -->
-        <thrustTopic>/thrusters/${name}/thrust</thrustTopic>
-        <!-- Thruster commmand input topic name -->
+         <thrusterName>${thruster_name}</thrusterName>
         <inputTopic>/thrusters/${name}/input</inputTopic>
-        <!-- Gain of the input command signal -->
-        <gain>1</gain>
-        <!-- Maximum allowed input value for the input signal for thruster unit -->
-        <clampMax>0</clampMax>
-        <!-- Minimum allowed value for the input signal for thruster unit -->
-        <clampMin>0</clampMin>
-        <!--
-        Value from 0 to 1 to set the efficiency of the output thrust force
-        Default value is 1.0
-        -->
-        <thrust_efficiency>1</thrust_efficiency>
-        <!--
-        Value from 0 to 1 to set the efficiency of the propeller as a factor
-        to be multiplied to the current value of the state variable at each
-        iteration.
-        Default value is 1.0
-        -->
-        <propeller_efficiency>1</propeller_efficiency>
-        <!-- Simple zero-order model -->
-        <dynamics>
-          <type>ZeroOrder</type>
-        </dynamics>
-        <!-- <dynamics>
-          <type>FirstOrder</type>
-          <timeConstant>0.0</timeConstant>
-        </dynamics>
-        <dynamics>
-          <type>Yoerger</type>
-          <alpha>0.0</alpha>
-          <beta>0.0</beta>
-        </dynamics>
-        <dynamics>
-          <type>Bessa</type>
-          <Jmsp>0.0</Jmsp>
-          <Kv1>0.0</Kv1>
-          <Kv2>0.0</Kv2>
-          <Kt>0.0</Kt>
-          <Rm>0.0</Rm>
-        </dynamics> -->
-        <conversion>
-          <type>Basic</type>
-          <rotorConstant>0.0</rotorConstant>
-        </conversion>
-        <!-- <conversion>
-          <type>Bessa</type>
-          <rotorConstantL>0.0</rotorConstantL>
-          <rotorConstantR>0.0</rotorConstantR>
-          <deltaL>0.0</deltaL>
-          <deltaR>0.0</deltaR>
-        </conversion>
-        <conversion>
-          <type>LinearInterp</type>
-          <inputValues>0 1 2 3</inputValues>
-          <outputValues>0 1 2 3</outputValues>
-        </conversion> -->
       </plugin>
     </gazebo>

Commit message: Fixed URDF for more DOF and better control

File: urdf/spaceship.urdf.xacro (robot description, xacro)
@@ -25,39 +25,51 @@
       </inertial>
     </link>
-    <xacro:thruster name="top_thruster" thruster_name="0">
-      <origin xyz="0 0 1.4" rpy="0 0 0"/>
+    <xacro:thruster name="top_left_front_thruster" thruster_name="0">
+      <origin xyz="3.8 3 4.6" rpy="0 0 0"/>
     </xacro:thruster>
-    <xacro:thruster name="bottom_thruster" thruster_name="1">
-      <origin xyz="0 0 -1.4" rpy="${pi} 0 0"/>
+    <xacro:thruster name="top_left_back_thruster" thruster_name="1">
+      <origin xyz="3.8 -3 4.6" rpy="0 0 0"/>
     </xacro:thruster>
-    <xacro:thruster name="front_thruster" thruster_name="2">
-      <origin xyz="0 1.4 0" rpy="${-pi/2} 0 0"/>
+    <xacro:thruster name="bottom_left_front_thruster" thruster_name="2">
+      <origin xyz="3.8 3 -4.6" rpy="0 ${pi} 0"/>
     </xacro:thruster>
-    <xacro:thruster name="back_thruster" thruster_name="3">
-      <origin xyz="0 -1.4 0" rpy="${pi/2} 0 0"/>
+    <xacro:thruster name="bottom_left_back_thruster" thruster_name="3">
+      <origin xyz="3.8 -3 -4.6" rpy="0 ${pi} 0"/>
     </xacro:thruster>
-    <xacro:thruster name="top_left_front_thruster" thruster_name="4">
-      <origin xyz="3.85 3 4.5" rpy="0 ${pi/2} 0"/>
+    <xacro:thruster name="top_right_front_thruster" thruster_name="4">
+      <origin xyz="-3.8 3 4.6" rpy="0 0 0"/>
     </xacro:thruster>
-    <xacro:thruster name="top_left_back_thruster" thruster_name="5">
-      <origin xyz="3.85 -3 4.5" rpy="0 ${pi/2} 0"/>
+    <xacro:thruster name="top_right_back_thruster" thruster_name="5">
+      <origin xyz="-3.8 -3 4.6" rpy="0 0 0"/>
     </xacro:thruster>
-    <xacro:thruster name="bottom_left_front_thruster" thruster_name="6">
-      <origin xyz="3.85 3 -4.5" rpy="0 ${pi/2} 0"/>
+    <xacro:thruster name="bottom_right_front_thruster" thruster_name="6">
+      <origin xyz="-3.8 3 -4.6" rpy="0 ${pi} 0"/>
     </xacro:thruster>
-    <xacro:thruster name="bottom_left_back_thruster" thruster_name="7">
-      <origin xyz="3.85 -3 -4.5" rpy="0 ${pi/2} 0"/>
+    <xacro:thruster name="bottom_right_back_thruster" thruster_name="7">
+      <origin xyz="-3.8 -3 -4.6" rpy="0 ${pi} 0"/>
     </xacro:thruster>
-    <xacro:thruster name="top_right_front_thruster" thruster_name="8">
-      <origin xyz="-3.85 3 4.5" rpy="0 ${-pi/2} 0"/>
+    <xacro:thruster name="side_top_left_front_thruster" thruster_name="8">
+      <origin xyz="3.8 3 4.5" rpy="0 ${pi/2} 0"/>
     </xacro:thruster>
-    <xacro:thruster name="top_right_back_thruster" thruster_name="9">
-      <origin xyz="-3.85 -3 4.5" rpy="0 ${-pi/2} 0"/>
+    <xacro:thruster name="side_top_left_back_thruster" thruster_name="9">
+      <origin xyz="3.8 -3 4.5" rpy="0 ${pi/2} 0"/>
     </xacro:thruster>
-    <xacro:thruster name="bottom_right_front_thruster" thruster_name="10">
-      <origin xyz="-3.85 3 -4.5" rpy="0 ${-pi/2} 0"/>
+    <xacro:thruster name="side_bottom_left_front_thruster" thruster_name="10">
+      <origin xyz="3.8 3 -4.5" rpy="0 ${pi/2} 0"/>
     </xacro:thruster>
-    <xacro:thruster name="bottom_right_back_thruster" thruster_name="11">
-      <origin xyz="-3.85 -3 -4.5" rpy="0 ${-pi/2} 0"/>
+    <xacro:thruster name="side_bottom_left_back_thruster" thruster_name="11">
+      <origin xyz="3.8 -3 -4.5" rpy="0 ${pi/2} 0"/>
+    </xacro:thruster>
+    <xacro:thruster name="side_top_right_front_thruster" thruster_name="12">
+      <origin xyz="-3.8 3 4.5" rpy="0 ${-pi/2} 0"/>
+    </xacro:thruster>
+    <xacro:thruster name="side_top_right_back_thruster" thruster_name="13">
+      <origin xyz="-3.8 -3 4.5" rpy="0 ${-pi/2} 0"/>
+    </xacro:thruster>
+    <xacro:thruster name="side_bottom_right_front_thruster" thruster_name="14">
+      <origin xyz="-3.8 3 -4.5" rpy="0 ${-pi/2} 0"/>
+    </xacro:thruster>
+    <xacro:thruster name="side_bottom_right_back_thruster" thruster_name="15">
+      <origin xyz="-3.8 -3 -4.5" rpy="0 ${-pi/2} 0"/>
     </xacro:thruster>
     <gazebo reference="base_link">

Commit message: Maximum DoF! :beers:

File: urdf/spaceship.urdf.xacro (robot description, xacro)
@@ -31,15 +31,15 @@
       <origin xyz="3.8 -3 4.6" rpy="0 0 0"/>
     </xacro:thruster>
-    <xacro:thruster name="bottom_left_front_thruster" thruster_name="2">
+    <xacro:thruster name="top_right_front_thruster" thruster_name="2">
+      <origin xyz="-3.8 3 4.6" rpy="0 0 0"/>
+    </xacro:thruster>
+    <xacro:thruster name="top_right_back_thruster" thruster_name="4">
+      <origin xyz="-3.8 -3 4.6" rpy="0 0 0"/>
+    </xacro:thruster>
+    <xacro:thruster name="bottom_left_front_thruster" thruster_name="5">
       <origin xyz="3.8 3 -4.6" rpy="0 ${pi} 0"/>
     </xacro:thruster>
-    <xacro:thruster name="bottom_left_back_thruster" thruster_name="3">
+    <xacro:thruster name="bottom_left_back_thruster" thruster_name="6">
       <origin xyz="3.8 -3 -4.6" rpy="0 ${pi} 0"/>
-    </xacro:thruster>
-    <xacro:thruster name="top_right_front_thruster" thruster_name="4">
-      <origin xyz="-3.8 3 4.6" rpy="0 0 0"/>
-    </xacro:thruster>
-    <xacro:thruster name="top_right_back_thruster" thruster_name="5">
-      <origin xyz="-3.8 -3 4.6" rpy="0 0 0"/>
     </xacro:thruster>
     <xacro:thruster name="bottom_right_front_thruster" thruster_name="6">
@@ -50,27 +50,60 @@
     </xacro:thruster>
     <xacro:thruster name="side_top_left_front_thruster" thruster_name="8">
-      <origin xyz="3.8 3 4.5" rpy="0 ${pi/2} 0"/>
+      <origin xyz="3.8 3 4.6" rpy="0 ${pi/2} 0"/>
     </xacro:thruster>
     <xacro:thruster name="side_top_left_back_thruster" thruster_name="9">
-      <origin xyz="3.8 -3 4.5" rpy="0 ${pi/2} 0"/>
+      <origin xyz="3.8 -3 4.6" rpy="0 ${pi/2} 0"/>
     </xacro:thruster>
     <xacro:thruster name="side_bottom_left_front_thruster" thruster_name="10">
-      <origin xyz="3.8 3 -4.5" rpy="0 ${pi/2} 0"/>
+      <origin xyz="3.8 3 -4.6" rpy="0 ${pi/2} 0"/>
     </xacro:thruster>
     <xacro:thruster name="side_bottom_left_back_thruster" thruster_name="11">
-      <origin xyz="3.8 -3 -4.5" rpy="0 ${pi/2} 0"/>
+      <origin xyz="3.8 -3 -4.6" rpy="0 ${pi/2} 0"/>
     </xacro:thruster>
     <xacro:thruster name="side_top_right_front_thruster" thruster_name="12">
-      <origin xyz="-3.8 3 4.5" rpy="0 ${-pi/2} 0"/>
+      <origin xyz="-3.8 3 4.6" rpy="0 ${-pi/2} 0"/>
     </xacro:thruster>
     <xacro:thruster name="side_top_right_back_thruster" thruster_name="13">
-      <origin xyz="-3.8 -3 4.5" rpy="0 ${-pi/2} 0"/>
+      <origin xyz="-3.8 -3 4.6" rpy="0 ${-pi/2} 0"/>
     </xacro:thruster>
     <xacro:thruster name="side_bottom_right_front_thruster" thruster_name="14">
-      <origin xyz="-3.8 3 -4.5" rpy="0 ${-pi/2} 0"/>
+      <origin xyz="-3.8 3 -4.6" rpy="0 ${-pi/2} 0"/>
     </xacro:thruster>
     <xacro:thruster name="side_bottom_right_back_thruster" thruster_name="15">
-      <origin xyz="-3.8 -3 -4.5" rpy="0 ${-pi/2} 0"/>
+      <origin xyz="-3.8 -3 -4.6" rpy="0 ${-pi/2} 0"/>
     </xacro:thruster>
+    <xacro:thruster name="front_top_left_thruster" thruster_name="16">
+      <origin xyz="3.8 3.1 4.6" rpy="${-pi/2} 0 0"/>
+    </xacro:thruster>
+    <xacro:thruster name="front_top_right_thruster" thruster_name="17">
+      <origin xyz="-3.8 3.1 4.6" rpy="${-pi/2} 0 0"/>
+    </xacro:thruster>
+    <xacro:thruster name="front_bottom_left_thruster" thruster_name="18">
+      <origin xyz="3.8 3.1 -4.6" rpy="${-pi/2} 0 0"/>
+    </xacro:thruster>
+    <xacro:thruster name="front_bottom_right_thruster" thruster_name="19">
+      <origin xyz="-3.8 3.1 -4.6" rpy="${-pi/2} 0 0"/>
+    </xacro:thruster>
+    <xacro:thruster name="back_top_left_thruster" thruster_name="20">
+      <origin xyz="3.8 -3.1 4.6" rpy="${pi/2} 0 0"/>
+    </xacro:thruster>
+    <xacro:thruster name="back_top_right_thruster" thruster_name="21">
+      <origin xyz="-3.8 -3.1 4.6" rpy="${pi/2} 0 0"/>
+    </xacro:thruster>
+    <xacro:thruster name="back_bottom_left_thruster" thruster_name="22">
+      <origin xyz="3.8 -3.1 -4.6" rpy="${pi/2} 0 0"/>
+    </xacro:thruster>
+    <xacro:thruster name="back_bottom_right_thruster" thruster_name="23">
+      <origin xyz="-3.8 -3.1 -4.6" rpy="${pi/2} 0 0"/>
+    </xacro:thruster>
+    <!-- <xacro:thruster name="top_left_back_thruster" thruster_name="1">
+      <origin xyz="3.8 -3 4.6" rpy="0 0 0"/>
+    </xacro:thruster>
+    <xacro:thruster name="top_right_front_thruster" thruster_name="2">
+      <origin xyz="-3.8 3 4.6" rpy="0 0 0"/>
+    </xacro:thruster>
+    <xacro:thruster name="top_right_back_thruster" thruster_name="4">
+      <origin xyz="-3.8 -3 4.6" rpy="0 0 0"/>
+    </xacro:thruster> -->
     <gazebo reference="base_link">
       <material>Gazebo/White</material>
